Commit message: Created Gazebo launch file

File: description/robot_core.xacro (robot description, xacro)
@@ -46,5 +46,9 @@
         <child link="left_wheel"/>
         <origin xyz="0 0.175 0" rpy="-${pi/2} 0 0"/>
-        <axis xyz="0 0 1"/>
+        <axis xyz="0 0 1">
+            <limit>
+                <effort>50000</effort> <!-- from <wheel_torque> in libgazebo_ros_diff_drive.so.-->
+            </limit>
+        </axis>
     </joint>
     <link name="left_wheel">
@@ -69,5 +73,9 @@
         <child link="right_wheel"/>
         <origin xyz="0 -0.175 0" rpy="${pi/2} 0 0"/>
-        <axis xyz="0 0 -1"/>
+        <axis xyz="0 0 -1">
+            <limit>
+                <effort>50000</effort> <!-- from <wheel_torque> in libgazebo_ros_diff_drive.so.-->
+            </limit>
+        </axis>
     </joint>
     <link name="right_wheel">

Commit message: Added Mount

File: description/robot_core.xacro (robot description, xacro)
@@ -37,5 +37,5 @@
             </geometry>
         </collision>
-        <xacro:inertial_box mass="0.5" x="0.5" y="0.3" z="0.15">
+        <xacro:inertial_box mass="0.5" x="0.3" y="0.3" z="0.15">
             <origin xyz="0.15 0 0.075" rpy="0 0 0"/>
         </xacro:inertial_box>
@@ -117,3 +117,27 @@
         </xacro:inertial_sphere>
     </link>
+    <!-- MOUNT -->
+    <joint name="mount_joint" type="fixed">
+        <parent link="chassis"/>
+        <child link="mount"/>
+        <origin xyz="0.125 0 0.15" rpy="0 0 0"/>
+    </joint>
+    <link name="mount">
+        <visual>
+            <origin xyz="0 0 0.5"/>
+            <geometry>
+                <cylinder radius="0.05" length="1"/>
+            </geometry>
+            <material name="white"/>
+        </visual>
+        <collision>
+            <origin xyz="0 0 0.5"/>
+            <geometry>
+                <cylinder radius="0.05" length="1"/>
+            </geometry>
+        </collision>
+        <xacro:inertial_cylinder mass="0.1" length="1" radius="0.05">
+            <origin xyz="0 0 0.5" rpy="0 0 0"/>
+        </xacro:inertial_cylinder>
+    </link>
 </robot>

Commit message: Djusted Mount and added Screen

File: description/robot_core.xacro (robot description, xacro)
@@ -121,11 +121,11 @@
         <parent link="chassis"/>
         <child link="mount"/>
-        <origin xyz="0.125 0 0.15" rpy="0 0 0"/>
+        <origin xyz="0.15 0 0.15" rpy="0 0 0"/>
     </joint>
     <link name="mount">
         <visual>
-            <origin xyz="0 0 0.5"/>
+            <origin xyz="0 0 0.4"/>
             <geometry>
-                <cylinder radius="0.05" length="1"/>
+                <cylinder radius="0.04" length="0.8"/>
             </geometry>
             <material name="white"/>
@@ -134,10 +134,34 @@
             <origin xyz="0 0 0.5"/>
             <geometry>
-                <cylinder radius="0.05" length="1"/>
+                <cylinder radius="0.04" length="0.8"/>
             </geometry>
         </collision>
-        <xacro:inertial_cylinder mass="0.1" length="1" radius="0.05">
-            <origin xyz="0 0 0.5" rpy="0 0 0"/>
+        <xacro:inertial_cylinder mass="0.1" length="0.8" radius="0.04">
+            <origin xyz="0 0 0" rpy="0 0 0"/>
         </xacro:inertial_cylinder>
     </link>
+    <!-- Screen -->
+    <joint name="screen_joint" type="fixed">
+        <parent link="mount"/>
+        <child link="screen"/>
+        <origin xyz="0.04 0 0.74"/>
+    </joint>
+    <link name="screen">
+        <visual>
+            <origin xyz="0.01 0 0"/>
+            <geometry>
+                <box size="0.02 0.2 0.14"/>
+            </geometry>
+            <material name="black"/>
+        </visual>
+        <collision>
+            <origin xyz="0.01 0 0"/>
+            <geometry>
+                <box size="0.02 0.2 0.14"/>
+            </geometry>
+        </collision>
+        <xacro:inertial_box mass="0.05" x="0.02" y="0.2" z="0.14">
+            <origin xyz="0.1 0 0" rpy="0 0 0"/>
+        </xacro:inertial_box>
+    </link>
 </robot>
