Commit message: Added Sensors with launch file and core updates.

File: description/robot.urdf.xacro (robot description, xacro)
@@ -3,3 +3,5 @@
     <xacro:include filename="robot_core.xacro" />
     <xacro:include filename="gazebo_control.xacro" />
+    <xacro:include filename="lidar.xacro" />
+    <xacro:include filename="camera.xacro" />
 </robot>

File: description/robot_core.xacro (robot description, xacro)
@@ -13,4 +13,7 @@
     <material name="black">
         <color rgba ="0 0 0 1" />
+    </material>
+    <material name="red">
+        <color rgba ="1 0 0 1" />
     </material>
     <!-- BASE LINK-->
@@ -132,5 +135,5 @@
         </visual>
         <collision>
-            <origin xyz="0 0 0.5"/>
+            <origin xyz="0 0 0.4"/>
             <geometry>
                 <cylinder radius="0.04" length="0.8"/>
@@ -138,5 +141,5 @@
         </collision>
         <xacro:inertial_cylinder mass="0.1" length="0.8" radius="0.04">
-            <origin xyz="0 0 0" rpy="0 0 0"/>
+            <origin xyz="0 0 0.4" rpy="0 0 0"/>
         </xacro:inertial_cylinder>
     </link>
@@ -162,6 +165,18 @@
         </collision>
         <xacro:inertial_box mass="0.05" x="0.02" y="0.2" z="0.14">
-            <origin xyz="0.1 0 0" rpy="0 0 0"/>
+            <origin xyz="0.01 0 0" rpy="0 0 0"/>
         </xacro:inertial_box>
     </link>
+    <gazebo reference="right_wheel">
+        <mu1>1.0</mu1>
+        <mu2>1.0</mu2>
+    </gazebo>
+    <gazebo reference="left_wheel">
+        <mu1>1.0</mu1>
+        <mu2>1.0</mu2>
+    </gazebo>
+    <gazebo reference="caster_wheel">
+        <mu1> 0.000001 </mu1>
+        <mu2> 0.000001 </mu2>
+    </gazebo>
 </robot>
